File: electronics/BLuesat power/1U power board.kicad_pcb (KiCad board)
At the start: 2 copper layers, 48.7 x 31.3 mm, 13 parts, among them J1 Conn_01x04_Male

Commit message: Overdue electronics changes
Parts:
- removed the REF** at (144.9, 77.8)
- removed the REF** at (144.7, 99.1)
- added REF**: MountingHole_3.2mm_M3, MountingHole:MountingHole_3.2mm_M3, F.Cu at (104.0, 74.0)
- added REF**: MountingHole_3.2mm_M3, MountingHole:MountingHole_3.2mm_M3, F.Cu at (104.0, 99.0)
- added REF**: MountingHole_3.2mm_M3, MountingHole:MountingHole_3.2mm_M3, F.Cu at (135.0, 74.0)
- added REF**: MountingHole_3.2mm_M3, MountingHole:MountingHole_3.2mm_M3, F.Cu at (135.0, 99.0)
- moved J1 6.00 mm to (111.0, 101.0)
Routing:
- net +3V3: track 20.0 -> 14.0 mm
- net +7.5V: track 29.3 -> 31.7 mm
Other:
- board size 48.7 x 31.3 mm -> 40.7 x 35.3 mm
