File: electronics/Sesnsor Board/Sensors.kicad_sch (KiCad schematic)
At the start: 16 parts, among them J2 JTAG, J3 UART, SW1 SW_Push, SW2 SW_Push, U1 ESP32-WROOM-E, U2 H3LIS100DLTR, Y1 32.768

Commit message: Batter Board almost finished
TODO
- Change mosfets&shunt resistor to new choice
- Adjust inductor for higher voltage
Parts:
- C_{X1}1: footprint (none) -> Capacitor_SMD:C_0805_2012Metric_Pad1.18x1.45mm_HandSolder
- R_{X}1: footprint (none) -> Resistor_SMD:R_0603_1608Metric_Pad0.98x0.95mm_HandSolder
Changed lines of the file:
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@@
       (effects (font (size 1.27 1.27)) (justify left))
     )
-    (property "Footprint" "" (id 2) (at 91.44 77.47 0)
+    (property "Footprint" "Resistor_SMD:R_0603_1608Metric_Pad0.98x0.95mm_HandSolder" (id 2) (at 91.44 77.47 0)
       (effects (font (size 1.27 1.27)) hide)
     )
@@
     (property "Reference" "C_{X1}1" (id 0) (at 83.8136 66.04 90))
     (property "Value" "25pF" (id 1) (at 83.8136 68.58 90))
-    (property "Footprint" "" (id 2) (at 83.82 72.39 0)
+    (property "Footprint" "Capacitor_SMD:C_0805_2012Metric_Pad1.18x1.45mm_HandSolder" (id 2) (at 83.82 72.39 0)
       (effects (font (size 1.27 1.27)) hide)
     )

Commit message: Long overdue commit
Connections:
- net I36: now also Board1.5 (D1)
- net I39: now also Board1.36 (D2)
- net IO26: now also Board1.12 (D5)
- net IO27: now also Board1.29 (D6)
Changed lines of the file:
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@@
+    (stroke (width 0) (type default) (color 0 0 0 0))
+  )
+  (wire (pts (xy 43.18 55.88) (xy 40.64 55.88))
     (stroke (width 0) (type default) (color 0 0 0 0))
   )
@@
     (stroke (width 0) (type default) (color 0 0 0 0))
   )
+  (wire (pts (xy 40.64 58.42) (xy 43.18 58.42))
+    (stroke (width 0) (type default) (color 0 0 0 0))
+  )
   (wire (pts (xy 119.38 50.8) (xy 119.38 46.99))
     (stroke (width 0) (type default) (color 0 0 0 0))
@@
     (stroke (width 0) (type default) (color 0 0 0 0))
   )
+  (wire (pts (xy 43.18 66.04) (xy 40.64 66.04))
+    (stroke (width 0) (type default) (color 0 0 0 0))
+  )
   (wire (pts (xy 260.35 113.03) (xy 265.43 113.03))
     (stroke (width 0) (type default) (color 0 0 0 0))
@@
     (stroke (width 0) (type default) (color 0 0 0 0))
   )
+  (wire (pts (xy 43.18 68.58) (xy 40.64 68.58))
+    (stroke (width 0) (type default) (color 0 0 0 0))
+  )
   (wire (pts (xy 129.54 105.41) (xy 114.3 105.41))
     (stroke (width 0) (type default) (color 0 0 0 0))
@@
     (effects (font (size 1.27 1.27)) (justify right bottom))
   )
+  (label "I36" (at 43.18 55.88 0)
+    (effects (font (size 1.27 1.27)) (justify left bottom))
+  )
   (label "IO32" (at 119.38 76.2 0)
     (effects (font (size 1.27 1.27)) (justify left bottom))
@@
     (effects (font (size 1.27 1.27)) (justify left bottom))
   )
+  (label "IO27" (at 43.18 68.58 0)
+    (effects (font (size 1.27 1.27)) (justify left bottom))
+  )
   (label "VCLK" (at 231.14 119.38 180)
     (effects (font (size 1.27 1.27)) (justify right bottom))
@@
     (effects (font (size 1.27 1.27)) (justify left bottom))
   )
+  (label "IO26" (at 43.18 66.04 0)
+    (effects (font (size 1.27 1.27)) (justify left bottom))
+  )
   (label "IO19" (at 205.74 59.69 180)
     (effects (font (size 1.27 1.27)) (justify right bottom))
@@
   (label "SCL1" (at 229.87 90.17 180)
     (effects (font (size 1.27 1.27)) (justify right bottom))
+  )
+  (label "I39" (at 43.18 58.42 0)
+    (effects (font (size 1.27 1.27)) (justify left bottom))
   )
   (label "IO23" (at 205.74 67.31 180)
@@
     (pin "1")
     (pin "2")
-  )
-  (symbol (lib_id "power:+3.3V") (at 231.14 110.49 90) (unit 1)
-    (in_bom yes) (on_board yes) (fields_autoplaced)
-    (property "Reference" "#PWR0122" (id 0) (at 234.95 110.49 0)
-      (effects (font (size 1.27 1.27)) hide)
-    )
-    (property "Value" "+3.3V" (id 1) (at 227.33 110.4899 90)
-      (effects (font (size 1.27 1.27)) (justify left))
-    )
-    (property "Footprint" "" (id 2) (at 231.14 110.49 0)
-      (effects (font (size 1.27 1.27)) hide)
-    )
-    (property "Datasheet" "" (id 3) (at 231.14 110.49 0)
-      (effects (font (size 1.27 1.27)) hide)
-    )
-    (pin "1")
   )
   (symbol (lib_id "power:GND") (at 265.43 100.33 90) (unit 1)
@@
     (pin "2")
   )
+  (symbol (lib_id "power:+5V") (at 231.14 110.49 90) (unit 1)
+    (in_bom yes) (on_board yes)
+    (property "Reference" "#PWR0122" (id 0) (at 234.95 110.49 0)
+      (effects (font (size 1.27 1.27)) hide)
+    )
+    (property "Value" "+5V" (id 1) (at 223.52 110.49 90)
+      (effects (font (size 1.27 1.27)) (justify right))
+    )
+    (property "Footprint" "" (id 2) (at 231.14 110.49 0)
+      (effects (font (size 1.27 1.27)) hide)
+    )
+    (property "Datasheet" "" (id 3) (at 231.14 110.49 0)
+      (effects (font (size 1.27 1.27)) hide)
+    )
+    (pin "1")
+  )
   (sheet (at 234.95 109.22) (size 25.4 16.51) (fields_autoplaced)
     (stroke (width 0.1524) (type solid) (color 0 0 0 0))
@@
       (reference "#PWR0121") (unit 1) (value "+5V") (footprint "")
     )
-    (path "/859cd8ac-164e-439b-b137-3920d71247d8"
-      (reference "#PWR0122") (unit 1) (value "+3.3V") (footprint "")
+    (path "/fde419c0-af52-4cb7-aafe-8315aab43c8d"
+      (reference "#PWR0122") (unit 1) (value "+5V") (footprint "")
     )
     (path "/f507e858-2bf9-43f8-8747-95a559eeac27"
